Commit message: wip

File: mobile_base_controller/zuuu_description/urdf/zuuu.urdf.xacro (robot description, xacro)
@@ -2,6 +2,6 @@
 <robot xmlns:xacro="http://www.ros.org/wiki/xacro" name="zuuu">
   <xacro:arg name="prefix" default=""/>
-  <xacro:arg name="model" default="" />
-  <xacro:arg name="use_gazebo" default="true"/>
+  <xacro:arg name="model" default="zuuu" />
+  <xacro:arg name="use_gazebo" default="false"/>
   <xacro:arg name="use_fake_components" default="true"/>
   <xacro:arg name="use_fixed_wheels" default="true"/>

File: mobile_base_controller/zuuu_description/urdf/zuuu_description.urdf.xacro (robot description, xacro)
@@ -44,5 +44,5 @@
     <!-- Robot Base -->
     <link name="base_link">
-      <!-- <visual>
+      <visual>
         <geometry>
           <cylinder radius="${base_radius}" length="${base_depth}"/>
@@ -51,11 +51,11 @@
           <color rgba="0 1.0 1.0 1.0"/>
         </material>
-      </visual> -->
-      <visual>
-        <origin xyz="0 0 ${(-base_top_height+base_depth/2)}" rpy="0 0 0"/>
-        <geometry>
-          <mesh filename="file://$(find zuuu_description)/meshes/reachy_mobile_pauvre.dae"/>
-        </geometry>
       </visual>
+      <!-- <visual> -->
+      <!--   <origin xyz="0 0 ${(-base_top_height+base_depth/2)}" rpy="0 0 0"/> -->
+      <!--   <geometry> -->
+      <!--     <mesh filename="package://zuuu_description/meshes/reachy_mobile_pauvre.dae"/> -->
+      <!--   </geometry> -->
+      <!-- </visual> -->
       <collision>
         <geometry>

File: reachy_description/urdf/reachy.urdf.xacro (robot description, xacro)
@@ -8,8 +8,36 @@
     <xacro:include filename="$(find reachy_description)/urdf/head.urdf.xacro"/>
     <xacro:include filename="$(find reachy_description)/urdf/orbita.urdf.xacro"/>
-    <link name="world"/>
-    <joint name="world_joint" type="fixed">
+    <!-- Add Zuuu mobile base -->
+    <!-- <xacro:include filename="$(find zuuu_description)/urdf/zuuu.urdf.xacro"/> -->
+  <xacro:arg name="prefix" default=""/>
+  <xacro:arg name="model" default="zuuu" />
+  <xacro:arg name="use_gazebo" default="false"/>
+  <xacro:arg name="use_fake_components" default="true"/>
+  <xacro:arg name="use_fixed_wheels" default="true"/>
+  <xacro:arg name="use_ros_control" default="true"/>
+    <!-- Import zuuu macro -->
+    <xacro:include filename="$(find zuuu_description)/urdf/zuuu_description.urdf.xacro"/>
+    <!-- Import Gazebo macro -->
+  <xacro:include filename="$(find zuuu_description)/urdf/zuuu.gazebo.xacro"/>
+  <!-- Import Zuuu ros2_control description -->
+  <xacro:include filename="$(find zuuu_description)/urdf/zuuu.ros2_control.xacro"/>
+  <xacro:zuuu
+      model="$(arg model)" prefix="$(arg prefix)">
+  </xacro:zuuu>
+  <xacro:if value="$(arg use_gazebo)">
+    <xacro:zuuu_gazebo model="$(arg model)" prefix="$(arg prefix)" />
+  </xacro:if>
+  <xacro:if value="$(arg use_ros_control)">
+    <xacro:zuuu_ros2_control model="$(arg model)" prefix="$(arg prefix)"/>
+  </xacro:if>
+    <!-- <link name="world"/> -->
+    <!-- <joint name="world_joint" type="fixed"> -->
+    <!--     <origin xyz="0 0 1.0" rpy="0 0 0"/> -->
+    <!--     <parent link="world"/> -->
+    <!--     <child link="torso"/> -->
+    <!-- </joint> -->
+    <joint name="base_joint" type="fixed">
         <origin xyz="0 0 1.0" rpy="0 0 0"/>
-        <parent link="world"/>
+        <parent link="base_link"/>
         <child link="torso"/>
     </joint>
