Commit message: seems ok

File: mobile_base_controller/zuuu_description/urdf/zuuu_description.urdf.xacro (robot description, xacro)
@@ -44,12 +44,12 @@
     <!-- Robot Base -->
     <link name="base_link">
-      <visual>
-        <geometry>
-          <cylinder radius="${base_radius}" length="${base_depth}"/>
-        </geometry>
-        <material name="Cyan">
-          <color rgba="0 1.0 1.0 1.0"/>
-        </material>
-      </visual>
+      <!-- <visual> -->
+      <!--   <geometry> -->
+      <!--     <cylinder radius="${base_radius}" length="${base_depth}"/> -->
+      <!--   </geometry> -->
+      <!--   <material name="Cyan"> -->
+      <!--     <color rgba="0 1.0 1.0 1.0"/> -->
+      <!--   </material> -->
+      <!-- </visual> -->
       <!-- <visual> -->
       <!--   <origin xyz="0 0 ${(-base_top_height+base_depth/2)}" rpy="0 0 0"/> -->
@@ -58,10 +58,23 @@
       <!--   </geometry> -->
       <!-- </visual> -->
-      <collision>
-        <geometry>
-          <cylinder radius="${base_radius}" length="${base_depth}"/>
-        </geometry>
-      </collision>
-      <xacro:cylinder_inertia m="20" r="${base_radius}" h="${base_depth}"/>
+	<visual>
+	  <origin xyz="0 0 0" rpy="0 0 0"/>
+	  <geometry>
+	    <mesh filename="file://$(find zuuu_description)/meshes/mobile_base_visual.dae" />
+	  </geometry>
+	</visual>
+	<collision>
+	  <origin xyz="0 0 0.13045" rpy="0 0 0"/>
+	  <geometry>
+	    <cylinder radius="0.245" length="0.2609"/>
+	  </geometry>
+	</collision>
+	<inertial>
+	  <origin xyz="0.008 -0.00048 0.112" rpy="0 0 0"/>
+	  <mass value="24.0"/>
+	  <inertia ixx="0.40791094" ixy="-0.00167148" ixz="-0.00178789"
+		   iyx="-0.00167148" iyy="0.4236827" iyz="0.00026596"
+		   izx="-0.00178789" izy="0.00026596" izz="0.70990763"/>
+	</inertial>
     </link>
     <!-- Wheels -->
@@ -76,11 +89,11 @@
           <material name="Bricks"></material>
         </visual> -->
-        <collision>
-          <origin xyz="0 0 0" rpy="${pi/2} 0 0"/>
-          <geometry>
-            <cylinder radius="${wheel_radius}" length="${wheel_width}"/>
-          </geometry>
-        </collision>
-        <xacro:cylinder_inertia m="0.5" r="${wheel_radius}" h="${wheel_width}"/>
+        <!-- <collision> -->
+        <!--   <origin xyz="0 0 0" rpy="${pi/2} 0 0"/> -->
+        <!--   <geometry> -->
+        <!--     <cylinder radius="${wheel_radius}" length="${wheel_width}"/> -->
+        <!--   </geometry> -->
+        <!-- </collision> -->
+        <!-- <xacro:cylinder_inertia m="0.5" r="${wheel_radius}" h="${wheel_width}"/> -->
       </link>
       <xacro:if value="$(arg use_fixed_wheels)">
@@ -150,10 +163,10 @@
         </geometry>
       </visual> -->
-      <collision>
-        <geometry>
-          <box size="0.1 0.1 0.1"/>
-        </geometry>
-      </collision>
-      <xacro:box_inertia m="0.1" w="0.1" d="0.1" h="0.1"/>
+      <!-- <collision> -->
+      <!--   <geometry> -->
+      <!--     <box size="0.1 0.1 0.1"/> -->
+      <!--   </geometry> -->
+      <!-- </collision> -->
+      <!-- <xacro:box_inertia m="0.1" w="0.1" d="0.1" h="0.1"/> -->
     </link>
     <joint name="imu_joint" type="fixed">
@@ -168,10 +181,10 @@
         <inertia ixx="0.001"  ixy="0"  ixz="0" iyy="0.001" iyz="0" izz="0.001" />
       </inertial>
-      <collision>
-        <origin xyz="0 0 0" rpy="0 0 0"/>
-        <geometry>
-          <cylinder radius="0.0508" length="0.055"/>
-        </geometry>
-      </collision>
+      <!-- <collision> -->
+      <!--   <origin xyz="0 0 0" rpy="0 0 0"/> -->
+      <!--   <geometry> -->
+      <!--     <cylinder radius="0.0508" length="0.055"/> -->
+      <!--   </geometry> -->
+      <!-- </collision> -->
       <!-- <visual>
         <origin xyz="0 0 0" rpy="0 0 0"/>

File: reachy_description/urdf/reachy.urdf.xacro (robot description, xacro)
@@ -38,7 +38,26 @@
     <!-- </joint> -->
     <joint name="base_joint" type="fixed">
-        <origin xyz="0 0 1.0" rpy="0 0 0"/>
+        <origin xyz="-0.006 0 1.0" rpy="0 0 0"/>
         <parent link="base_link"/>
         <child link="torso"/>
+    </joint>
+    <link name="bar_link">
+      <visual name="">
+        <origin xyz="0.0 0.0 0.6125" rpy="0.0 0.0 0.0"/>
+            <geometry>
+              <cylinder radius="0.02" length="0.775"/>
+            </geometry>
+      </visual>
+      <collision>
+        <origin xyz="0.0 0.0 0.6125" rpy="0.0 0.0 0.0"/>
+            <geometry>
+              <cylinder radius="0.02" length="0.775"/>
+            </geometry>
+      </collision>
+    </link>
+    <joint name="bar_joint" type="fixed">
+        <origin xyz="-0.130 0 0.0" rpy="0 0 0"/>
+        <parent link="base_link"/>
+        <child link="bar_link"/>
     </joint>
     <link name="torso">

Commit message: update lidar and wheels

File: mobile_base_controller/zuuu_description/urdf/zuuu_description.urdf.xacro (robot description, xacro)
@@ -64,8 +64,14 @@
 	  </geometry>
 	</visual>
+	<!-- <collision> -->
+	<!--   <origin xyz="0 0 0.13045" rpy="0 0 0"/> -->
+	<!--   <geometry> -->
+	<!--     <cylinder radius="0.245" length="0.2609"/> -->
+	<!--   </geometry> -->
+	<!-- </collision> -->
 	<collision>
-	  <origin xyz="0 0 0.13045" rpy="0 0 0"/>
+	  <origin xyz="0 0 0.160" rpy="0 0 0"/>
 	  <geometry>
-	    <cylinder radius="0.245" length="0.2609"/>
+	    <cylinder radius="0.245" length="0.220"/>
 	  </geometry>
 	</collision>
@@ -81,5 +87,5 @@
     <xacro:macro name="wheel" params="prefix yaw_angle">
       <link name="${prefix}_link">
-        <!-- <visual>
+        <visual>
           <origin xyz="0 0 0" rpy="${pi/2} 0 0"/>
           <geometry>
@@ -88,12 +94,12 @@
           </geometry>
           <material name="Bricks"></material>
-        </visual> -->
-        <!-- <collision> -->
-        <!--   <origin xyz="0 0 0" rpy="${pi/2} 0 0"/> -->
-        <!--   <geometry> -->
-        <!--     <cylinder radius="${wheel_radius}" length="${wheel_width}"/> -->
-        <!--   </geometry> -->
-        <!-- </collision> -->
-        <!-- <xacro:cylinder_inertia m="0.5" r="${wheel_radius}" h="${wheel_width}"/> -->
+        </visual>
+        <collision>
+          <origin xyz="0 0 0" rpy="${pi/2} 0 0"/>
+          <geometry>
+            <cylinder radius="${wheel_radius}" length="${wheel_width}"/>
+          </geometry>
+        </collision>
+        <xacro:cylinder_inertia m="0.5" r="${wheel_radius}" h="${wheel_width}"/>
       </link>
       <xacro:if value="$(arg use_fixed_wheels)">
@@ -101,5 +107,5 @@
             <parent link="base_link"/>
             <child link="${prefix}_link"/>
-            <origin xyz="${wheel_radial_dist*cos(yaw_angle)} ${-wheel_radial_dist*sin(yaw_angle)} ${-((base_top_height-base_depth/2)- wheel_radius)}" rpy="0 0 ${pi/2-yaw_angle}"/>
+            <origin xyz="${(wheel_radial_dist+wheel_width/2)*cos(yaw_angle)} ${-(wheel_radial_dist+wheel_width/2)*sin(yaw_angle)} ${(wheel_radius)}" rpy="0 0 ${pi/2-yaw_angle}"/>
             <axis xyz="0 1 0"/>
             <joint_properties damping="${global_damping}" friction="${global_friction}"/>
@@ -121,5 +127,6 @@
           <parent link="base_link"/>
           <child link="${prefix}_link"/>
-          <origin xyz="${wheel_radial_dist*cos(yaw_angle)} ${-wheel_radial_dist*sin(yaw_angle)} ${-((base_top_height-base_depth/2)- wheel_radius)}" rpy="0 0 ${pi/2-yaw_angle}"/>
+          <!-- <origin xyz="${wheel_radial_dist*cos(yaw_angle)} ${-wheel_radial_dist*sin(yaw_angle)} ${-((base_top_height-base_depth/2)- wheel_radius)}" rpy="0 0 ${pi/2-yaw_angle}"/> -->
+	  <origin xyz="${(wheel_radial_dist+wheel_width/2)*cos(yaw_angle)} ${-(wheel_radial_dist+wheel_width/2)*sin(yaw_angle)} ${(wheel_radius)}" rpy="0 0 ${pi/2-yaw_angle}"/>
           <axis xyz="0 1 0"/>
           <joint_properties damping="${global_damping}" friction="${global_friction}"/>
@@ -199,5 +206,6 @@
       <!-- <origin xyz="0.155 0 0.2" rpy="0 0 0"/> -->
       <!-- The -0.0129 were added on 22 pril 2022 for the second version of Zuuu. The 2mm pads are not taken into account -->
-      <origin xyz="0.155 0 ${-(base_top_height-base_depth/2)+base_top_height+0.105 -0.0129}" rpy="0 0 0"/>
+      <!-- <origin xyz="0.155 0 ${-(base_top_height-base_depth/2)+base_top_height+0.105 -0.0129}" rpy="0 0 0"/> -->
+      <origin xyz="0.175 0 0.24" rpy="0 0 0"/>
     </joint>
     <link name="camera_link">

Commit message: update lidar

File: mobile_base_controller/zuuu_description/urdf/zuuu_description.urdf.xacro (robot description, xacro)
@@ -71,7 +71,7 @@
 	<!-- </collision> -->
 	<collision>
-	  <origin xyz="0 0 0.160" rpy="0 0 0"/>
+	  <origin xyz="0 0 0.145" rpy="0 0 0"/>
 	  <geometry>
-	    <cylinder radius="0.245" length="0.220"/>
+	    <cylinder radius="0.245" length="0.19"/>
 	  </geometry>
 	</collision>
@@ -188,10 +188,10 @@
         <inertia ixx="0.001"  ixy="0"  ixz="0" iyy="0.001" iyz="0" izz="0.001" />
       </inertial>
-      <!-- <collision> -->
-      <!--   <origin xyz="0 0 0" rpy="0 0 0"/> -->
-      <!--   <geometry> -->
-      <!--     <cylinder radius="0.0508" length="0.055"/> -->
-      <!--   </geometry> -->
-      <!-- </collision> -->
+      <collision>
+        <origin xyz="0 0 0" rpy="0 0 0"/>
+        <geometry>
+          <cylinder radius="0.035" length="0.035"/>
+        </geometry>
+      </collision>
       <!-- <visual>
         <origin xyz="0 0 0" rpy="0 0 0"/>
@@ -207,5 +207,5 @@
       <!-- The -0.0129 were added on 22 pril 2022 for the second version of Zuuu. The 2mm pads are not taken into account -->
       <!-- <origin xyz="0.155 0 ${-(base_top_height-base_depth/2)+base_top_height+0.105 -0.0129}" rpy="0 0 0"/> -->
-      <origin xyz="0.175 0 0.24" rpy="0 0 0"/>
+      <origin xyz="0.184 0 0.24" rpy="0 0 0"/>
     </joint>
     <link name="camera_link">

Commit message: elevating the LIDAR to avoid self collision

File: mobile_base_controller/zuuu_description/urdf/zuuu_description.urdf.xacro (robot description, xacro)
@@ -207,5 +207,5 @@
       <!-- The -0.0129 were added on 22 pril 2022 for the second version of Zuuu. The 2mm pads are not taken into account -->
       <!-- <origin xyz="0.155 0 ${-(base_top_height-base_depth/2)+base_top_height+0.105 -0.0129}" rpy="0 0 0"/> -->
-      <origin xyz="0.184 0 0.24" rpy="0 0 0"/>
+      <origin xyz="0.184 0 0.25" rpy="0 0 0"/>
     </joint>
     <link name="camera_link">
